Commit message: Estimator changed to 1st order, force control in the xy plane

File: uav-cable-suspended-robots/uav-cable-suspended-robots-ros-pkg/urdf/licasa1_sensor_wall.urdf.xacro (robot description, xacro)
@@ -4,5 +4,5 @@
   <link name="world" />
   <joint name="sensor_wall_base_joint" type="fixed">
-    <origin xyz="2.5 0 0.05"/>
+    <origin xyz="2.5 0 0.05" rpy="0 0 0"/>
     <parent link="world"/>
     <child link="sensor_wall_base"/>

Commit message: increased p gain of the shoulder z revolute joint controller

File: uav-cable-suspended-robots/uav-cable-suspended-robots-ros-pkg/urdf/licasa1_sensor_wall.urdf.xacro (robot description, xacro)
@@ -4,5 +4,5 @@
   <link name="world" />
   <joint name="sensor_wall_base_joint" type="fixed">
-    <origin xyz="2.5 0 0.05" rpy="0 0 0"/>
+    <origin xyz="2.5 0 0.05" rpy="0 0 0.75"/>
     <parent link="world"/>
     <child link="sensor_wall_base"/>
