Commit message: removed unused files

File: rotors_simulator/rotors_description/urdf/licasa1.xacro (robot description, xacro)
@@ -143,46 +143,4 @@
     <xacro:insert_block name="rotor_inertia" />
   </xacro:vertical_rotor>
-  <!-- <xacro:vertical_rotor
-    robot_namespace="${namespace}"
-    suffix="right"
-    direction="ccw"
-    motor_constant="${motor_constant}"
-    moment_constant="${moment_constant}"
-    parent="${namespace}/base_link"
-    mass_rotor="${mass_rotor}"
-    radius_rotor="${radius_rotor}"
-    time_constant_up="${time_constant_up}"
-    time_constant_down="${time_constant_down}"
-    max_rot_velocity="${max_rot_velocity}"
-    motor_number="4"
-    rotor_drag_coefficient="${rotor_drag_coefficient}"
-    rolling_moment_coefficient="${rolling_moment_coefficient}"
-    color="Blue"
-    use_own_mesh="false"
-    mesh="">
-    <origin xyz="0 -${arm_length} ${rotor_offset_top}" rpy="0 0 0" />
-    <xacro:insert_block name="rotor_inertia" />
-  </xacro:vertical_rotor>
-  <xacro:vertical_rotor
-    robot_namespace="${namespace}"
-    suffix="front_right"
-    direction="cw"
-    motor_constant="${motor_constant}"
-    moment_constant="${moment_constant}"
-    parent="${namespace}/base_link"
-    mass_rotor="${mass_rotor}"
-    radius_rotor="${radius_rotor}"
-    time_constant_up="${time_constant_up}"
-    time_constant_down="${time_constant_down}"
-    max_rot_velocity="${max_rot_velocity}"
-    motor_number="5"
-    rotor_drag_coefficient="${rotor_drag_coefficient}"
-    rolling_moment_coefficient="${rolling_moment_coefficient}"
-    color="Red"
-    use_own_mesh="false"
-    mesh="">
-    <origin xyz="${cos30*arm_length} -${sin30*arm_length} ${rotor_offset_top}" rpy="0 0 0" />
-    <xacro:insert_block name="rotor_inertia" />
-  </xacro:vertical_rotor> -->
   <!-- Import Transmissions -->
   <xacro:include filename="$(find uav-cable-suspended-robots-ros-pkg)/urdf/licasa1.transmission.xacro" />

Commit message: Added estimator based hierarchical controller for the UAV

File: rotors_simulator/rotors_description/urdf/licasa1.xacro (robot description, xacro)
@@ -100,5 +100,5 @@
     use_own_mesh="false"
     mesh="">
-    <origin xyz="0 ${arm_length} ${rotor_offset_top}" rpy="0 0 0" />
+    <origin xyz="0 -${arm_length} ${rotor_offset_top}" rpy="0 0 0" />
     <xacro:insert_block name="rotor_inertia" />
   </xacro:vertical_rotor>
@@ -117,5 +117,5 @@
     rotor_drag_coefficient="${rotor_drag_coefficient}"
     rolling_moment_coefficient="${rolling_moment_coefficient}"
-    color="Blue"
+    color="Green"
     use_own_mesh="false"
     mesh="">
@@ -137,8 +137,8 @@
     rotor_drag_coefficient="${rotor_drag_coefficient}"
     rolling_moment_coefficient="${rolling_moment_coefficient}"
-    color="Blue"
+    color="Yellow"
     use_own_mesh="false"
     mesh="">
-    <origin xyz="0 -${arm_length} ${rotor_offset_top}" rpy="0 0 0" />
+    <origin xyz="0 ${arm_length} ${rotor_offset_top}" rpy="0 0 0" />
     <xacro:insert_block name="rotor_inertia" />
   </xacro:vertical_rotor>
@@ -281,10 +281,10 @@
       </geometry>
     </visual>
-    <collision>
+    <!-- <collision>
       <origin xyz="0 0 0"/>
       <geometry>
         <mesh filename="package://uav-cable-suspended-robots-ros-pkg/mesh/licas/Shoulder_Pitch_Structure.dae" scale=".001 .001 .001"/>
       </geometry>
-    </collision>
+    </collision> -->
   </link>
   <!-- LEFT ARM-->
@@ -309,10 +309,10 @@
       </geometry>
     </visual>
-    <collision>
+    <!-- <collision>
       <origin xyz="0 0.04 0"/>
       <geometry>
         <mesh filename="package://uav-cable-suspended-robots-ros-pkg/mesh/licas/Shoulder_Roll_Structure_Left.dae" scale=".001 .001 .001"/>
       </geometry>
-    </collision>
+    </collision> -->
   </link>
   <joint name="LiCAS_A1_q1_2" type="revolute">
@@ -336,10 +336,10 @@
       </geometry>
     </visual>
-    <collision>
+    <!-- <collision>
       <origin xyz="0 0 0"/>
       <geometry>
         <mesh filename="package://uav-cable-suspended-robots-ros-pkg/mesh/licas/Assembly_Shoulder_Yaw_Structure.dae" scale=".001 .001 .001"/>
       </geometry>
-    </collision>
+    </collision> -->
   </link>
   <joint name="LiCAS_A1_q1_3" type="revolute">
@@ -363,10 +363,10 @@
       </geometry>
     </visual>
-    <collision>
+    <!-- <collision>
       <origin xyz="0 0 -0.132"/>
       <geometry>
         <mesh filename="package://uav-cable-suspended-robots-ros-pkg/mesh/licas/Elbow_Pitch_Structure_Left_Cut.dae" scale=".001 .001 .001"/>
       </geometry>
-    </collision>
+    </collision> -->
   </link>
   <joint name="LiCAS_A1_q1_4" type="revolute">
@@ -390,10 +390,10 @@
       </geometry>
     </visual>
-    <collision>
+    <!-- <collision>
       <origin xyz="0 0 0"/>
       <geometry>
         <mesh filename="package://uav-cable-suspended-robots-ros-pkg/mesh/licas/Forearm_Link_with_Gripper_Servo.dae" scale=".001 .001 .001"/>
       </geometry>
-    </collision>
+    </collision> -->
   </link>
   <!-- RIGHT ARM-->
@@ -418,10 +418,10 @@
       </geometry>
     </visual>
-    <collision>
+    <!-- <collision>
       <origin xyz="0 -0.04 0"/>
       <geometry>
         <mesh filename="package://uav-cable-suspended-robots-ros-pkg/mesh/licas/Shoulder_Roll_Structure_Right.dae" scale=".001 .001 .001"/>
       </geometry>
-    </collision>
+    </collision> -->
   </link>
   <joint name="LiCAS_A1_q2_2" type="revolute">
@@ -445,10 +445,10 @@
       </geometry>
     </visual>
-    <collision>
+    <!-- <collision>
       <origin xyz="0 0 0"/>
       <geometry>
         <mesh filename="package://uav-cable-suspended-robots-ros-pkg/mesh/licas/Assembly_Shoulder_Yaw_Structure.dae" scale=".001 .001 .001"/>
       </geometry>
-    </collision>
+    </collision> -->
   </link>
   <joint name="LiCAS_A1_q2_3" type="revolute">
@@ -472,10 +472,10 @@
       </geometry>
     </visual>
-    <collision>
+    <!-- <collision>
       <origin xyz="0 0 -0.132"/>
       <geometry>
         <mesh filename="package://uav-cable-suspended-robots-ros-pkg/mesh/licas/Elbow_Pitch_Structure_Right_Cut.dae" scale=".001 .001 .001"/>
       </geometry>
-    </collision>
+    </collision> -->
   </link>
   <joint name="LiCAS_A1_q2_4" type="revolute">
@@ -499,10 +499,10 @@
       </geometry>
     </visual>
-    <collision>
+    <!-- <collision>
       <origin xyz="0 0 0"/>
       <geometry>
         <mesh filename="package://uav-cable-suspended-robots-ros-pkg/mesh/licas/Forearm_Link_with_Gripper_Servo.dae" scale=".001 .001 .001"/>
       </geometry>
-    </collision>
+    </collision> -->
   </link>
   <!-- END EFFECTORS -->

Commit message: Revert "Added estimator based hierarchical controller for the UAV"
This reverts commit 7a6c417790cc4578d693dd4784fd24e904085c92.

File: rotors_simulator/rotors_description/urdf/licasa1.xacro (robot description, xacro)
@@ -100,5 +100,5 @@
     use_own_mesh="false"
     mesh="">
-    <origin xyz="0 -${arm_length} ${rotor_offset_top}" rpy="0 0 0" />
+    <origin xyz="0 ${arm_length} ${rotor_offset_top}" rpy="0 0 0" />
     <xacro:insert_block name="rotor_inertia" />
   </xacro:vertical_rotor>
@@ -117,5 +117,5 @@
     rotor_drag_coefficient="${rotor_drag_coefficient}"
     rolling_moment_coefficient="${rolling_moment_coefficient}"
-    color="Green"
+    color="Blue"
     use_own_mesh="false"
     mesh="">
@@ -137,8 +137,8 @@
     rotor_drag_coefficient="${rotor_drag_coefficient}"
     rolling_moment_coefficient="${rolling_moment_coefficient}"
-    color="Yellow"
+    color="Blue"
     use_own_mesh="false"
     mesh="">
-    <origin xyz="0 ${arm_length} ${rotor_offset_top}" rpy="0 0 0" />
+    <origin xyz="0 -${arm_length} ${rotor_offset_top}" rpy="0 0 0" />
     <xacro:insert_block name="rotor_inertia" />
   </xacro:vertical_rotor>
@@ -281,10 +281,10 @@
       </geometry>
     </visual>
-    <!-- <collision>
+    <collision>
       <origin xyz="0 0 0"/>
       <geometry>
         <mesh filename="package://uav-cable-suspended-robots-ros-pkg/mesh/licas/Shoulder_Pitch_Structure.dae" scale=".001 .001 .001"/>
       </geometry>
-    </collision> -->
+    </collision>
   </link>
   <!-- LEFT ARM-->
@@ -309,10 +309,10 @@
       </geometry>
     </visual>
-    <!-- <collision>
+    <collision>
       <origin xyz="0 0.04 0"/>
       <geometry>
         <mesh filename="package://uav-cable-suspended-robots-ros-pkg/mesh/licas/Shoulder_Roll_Structure_Left.dae" scale=".001 .001 .001"/>
       </geometry>
-    </collision> -->
+    </collision>
   </link>
   <joint name="LiCAS_A1_q1_2" type="revolute">
@@ -336,10 +336,10 @@
       </geometry>
     </visual>
-    <!-- <collision>
+    <collision>
       <origin xyz="0 0 0"/>
       <geometry>
         <mesh filename="package://uav-cable-suspended-robots-ros-pkg/mesh/licas/Assembly_Shoulder_Yaw_Structure.dae" scale=".001 .001 .001"/>
       </geometry>
-    </collision> -->
+    </collision>
   </link>
   <joint name="LiCAS_A1_q1_3" type="revolute">
@@ -363,10 +363,10 @@
       </geometry>
     </visual>
-    <!-- <collision>
+    <collision>
       <origin xyz="0 0 -0.132"/>
       <geometry>
         <mesh filename="package://uav-cable-suspended-robots-ros-pkg/mesh/licas/Elbow_Pitch_Structure_Left_Cut.dae" scale=".001 .001 .001"/>
       </geometry>
-    </collision> -->
+    </collision>
   </link>
   <joint name="LiCAS_A1_q1_4" type="revolute">
@@ -390,10 +390,10 @@
       </geometry>
     </visual>
-    <!-- <collision>
+    <collision>
       <origin xyz="0 0 0"/>
       <geometry>
         <mesh filename="package://uav-cable-suspended-robots-ros-pkg/mesh/licas/Forearm_Link_with_Gripper_Servo.dae" scale=".001 .001 .001"/>
       </geometry>
-    </collision> -->
+    </collision>
   </link>
   <!-- RIGHT ARM-->
@@ -418,10 +418,10 @@
       </geometry>
     </visual>
-    <!-- <collision>
+    <collision>
       <origin xyz="0 -0.04 0"/>
       <geometry>
         <mesh filename="package://uav-cable-suspended-robots-ros-pkg/mesh/licas/Shoulder_Roll_Structure_Right.dae" scale=".001 .001 .001"/>
       </geometry>
-    </collision> -->
+    </collision>
   </link>
   <joint name="LiCAS_A1_q2_2" type="revolute">
@@ -445,10 +445,10 @@
       </geometry>
     </visual>
-    <!-- <collision>
+    <collision>
       <origin xyz="0 0 0"/>
       <geometry>
         <mesh filename="package://uav-cable-suspended-robots-ros-pkg/mesh/licas/Assembly_Shoulder_Yaw_Structure.dae" scale=".001 .001 .001"/>
       </geometry>
-    </collision> -->
+    </collision>
   </link>
   <joint name="LiCAS_A1_q2_3" type="revolute">
@@ -472,10 +472,10 @@
       </geometry>
     </visual>
-    <!-- <collision>
+    <collision>
       <origin xyz="0 0 -0.132"/>
       <geometry>
         <mesh filename="package://uav-cable-suspended-robots-ros-pkg/mesh/licas/Elbow_Pitch_Structure_Right_Cut.dae" scale=".001 .001 .001"/>
       </geometry>
-    </collision> -->
+    </collision>
   </link>
   <joint name="LiCAS_A1_q2_4" type="revolute">
@@ -499,10 +499,10 @@
       </geometry>
     </visual>
-    <!-- <collision>
+    <collision>
       <origin xyz="0 0 0"/>
       <geometry>
         <mesh filename="package://uav-cable-suspended-robots-ros-pkg/mesh/licas/Forearm_Link_with_Gripper_Servo.dae" scale=".001 .001 .001"/>
       </geometry>
-    </collision> -->
+    </collision>
   </link>
   <!-- END EFFECTORS -->

Commit message: Added launchpad, lift off sequence and sensorized wall

File: rotors_simulator/rotors_description/urdf/licasa1.xacro (robot description, xacro)
@@ -23,6 +23,6 @@
   <xacro:property name="mesh_file" value="package://rotors_description/meshes/firefly.dae" />
   <xacro:property name="mass" value="20.269" /> <!-- 1.5 [kg] -->
-  <xacro:property name="body_width" value="0.3" /> <!-- 0.1 [m] -->
-  <xacro:property name="body_height" value="0.48" /> <!-- 0.16 [m] -->
+  <xacro:property name="body_width" value="0.6" /> <!-- 0.1 [m] -->
+  <xacro:property name="body_height" value="0.24" /> <!-- 0.16 [m] -->
   <xacro:property name="mass_rotor" value="0.0001" /> <!-- 0.005 [kg] -->
   <xacro:property name="arm_length" value="0.645" /> <!-- 0.215 [m] -->
@@ -281,10 +281,10 @@
       </geometry>
     </visual>
-    <!-- <collision>
+    <collision>
       <origin xyz="0 0 0"/>
       <geometry>
         <mesh filename="package://uav-cable-suspended-robots-ros-pkg/mesh/licas/Shoulder_Pitch_Structure.dae" scale=".001 .001 .001"/>
       </geometry>
-    </collision> -->
+    </collision>
   </link>
   <!-- LEFT ARM-->
@@ -309,10 +309,10 @@
       </geometry>
     </visual>
-    <!-- <collision>
+    <collision>
       <origin xyz="0 0.04 0"/>
       <geometry>
         <mesh filename="package://uav-cable-suspended-robots-ros-pkg/mesh/licas/Shoulder_Roll_Structure_Left.dae" scale=".001 .001 .001"/>
       </geometry>
-    </collision> -->
+    </collision>
   </link>
   <joint name="LiCAS_A1_q1_2" type="revolute">
@@ -336,10 +336,10 @@
       </geometry>
     </visual>
-    <!-- <collision>
+    <collision>
       <origin xyz="0 0 0"/>
       <geometry>
         <mesh filename="package://uav-cable-suspended-robots-ros-pkg/mesh/licas/Assembly_Shoulder_Yaw_Structure.dae" scale=".001 .001 .001"/>
       </geometry>
-    </collision> -->
+    </collision>
   </link>
   <joint name="LiCAS_A1_q1_3" type="revolute">
@@ -363,10 +363,10 @@
       </geometry>
     </visual>
-    <!-- <collision>
+    <collision>
       <origin xyz="0 0 -0.132"/>
       <geometry>
         <mesh filename="package://uav-cable-suspended-robots-ros-pkg/mesh/licas/Elbow_Pitch_Structure_Left_Cut.dae" scale=".001 .001 .001"/>
       </geometry>
-    </collision> -->
+    </collision>
   </link>
   <joint name="LiCAS_A1_q1_4" type="revolute">
@@ -390,10 +390,10 @@
       </geometry>
     </visual>
-    <!-- <collision>
+    <collision>
       <origin xyz="0 0 0"/>
       <geometry>
         <mesh filename="package://uav-cable-suspended-robots-ros-pkg/mesh/licas/Forearm_Link_with_Gripper_Servo.dae" scale=".001 .001 .001"/>
       </geometry>
-    </collision> -->
+    </collision>
   </link>
   <!-- RIGHT ARM-->
@@ -418,10 +418,10 @@
       </geometry>
     </visual>
-    <!-- <collision>
+    <collision>
       <origin xyz="0 -0.04 0"/>
       <geometry>
         <mesh filename="package://uav-cable-suspended-robots-ros-pkg/mesh/licas/Shoulder_Roll_Structure_Right.dae" scale=".001 .001 .001"/>
       </geometry>
-    </collision> -->
+    </collision>
   </link>
   <joint name="LiCAS_A1_q2_2" type="revolute">
@@ -445,10 +445,10 @@
       </geometry>
     </visual>
-    <!-- <collision>
+    <collision>
       <origin xyz="0 0 0"/>
       <geometry>
         <mesh filename="package://uav-cable-suspended-robots-ros-pkg/mesh/licas/Assembly_Shoulder_Yaw_Structure.dae" scale=".001 .001 .001"/>
       </geometry>
-    </collision> -->
+    </collision>
   </link>
   <joint name="LiCAS_A1_q2_3" type="revolute">
@@ -472,10 +472,10 @@
       </geometry>
     </visual>
-    <!-- <collision>
+    <collision>
       <origin xyz="0 0 -0.132"/>
       <geometry>
         <mesh filename="package://uav-cable-suspended-robots-ros-pkg/mesh/licas/Elbow_Pitch_Structure_Right_Cut.dae" scale=".001 .001 .001"/>
       </geometry>
-    </collision> -->
+    </collision>
   </link>
   <joint name="LiCAS_A1_q2_4" type="revolute">
@@ -499,10 +499,10 @@
       </geometry>
     </visual>
-    <!-- <collision>
+    <collision>
       <origin xyz="0 0 0"/>
       <geometry>
         <mesh filename="package://uav-cable-suspended-robots-ros-pkg/mesh/licas/Forearm_Link_with_Gripper_Servo.dae" scale=".001 .001 .001"/>
       </geometry>
-    </collision> -->
+    </collision>
   </link>
   <!-- END EFFECTORS -->
@@ -531,5 +531,92 @@
     </inertial>
   </link>
-  <!-- Include MY URDF Files
-  <xacro:include filename="$(find cable-suspended-robots-ros-pkg)/urdf/licasa1.urdf.xacro" /> -->
+  <!-- Enable the Joint Feedback -->
+    <!-- The ft_sensor plugin -->
+  <!-- <gazebo reference="LiCAS_A1_q1_1">
+    <provideFeedback>true</provideFeedback>
+  </gazebo>
+  <gazebo>
+    <plugin name="LiCAS_A1_q1_1_sensor" filename="libgazebo_ros_ft_sensor.so">
+      <updateRate>100.0</updateRate>
+      <topicName>LiCAS_A1_q1_1_sensor</topicName>
+      <jointName>LiCAS_A1_q1_1</jointName>
+    </plugin>
+  </gazebo> -->
+  <!-- <gazebo reference="LiCAS_A1_q1_2">
+    <provideFeedback>true</provideFeedback>
+  </gazebo>
+  <gazebo>
+    <plugin name="LiCAS_A1_q1_2_sensor" filename="libgazebo_ros_ft_sensor.so">
+      <updateRate>100.0</updateRate>
+      <topicName>LiCAS_A1_q1_2_sensor</topicName>
+      <jointName>LiCAS_A1_q1_2</jointName>
+    </plugin>
+  </gazebo> -->
+  <!-- <gazebo reference="LiCAS_A1_q1_3">
+    <provideFeedback>true</provideFeedback>
+  </gazebo>
+  <gazebo>
+    <plugin name="LiCAS_A1_q1_3_sensor" filename="libgazebo_ros_ft_sensor.so">
+      <updateRate>100.0</updateRate>
+      <topicName>LiCAS_A1_q1_3_sensor</topicName>
+      <jointName>LiCAS_A1_q1_3</jointName>
+    </plugin>
+  </gazebo> -->
+  <!-- <gazebo reference="LiCAS_A1_q1_4">
+    <provideFeedback>true</provideFeedback>
+  </gazebo>
+  <gazebo>
+    <plugin name="LiCAS_A1_q1_4_sensor" filename="libgazebo_ros_ft_sensor.so">
+      <updateRate>100.0</updateRate>
+      <topicName>LiCAS_A1_q1_4_sensor</topicName>
+      <jointName>LiCAS_A1_q1_4</jointName>
+    </plugin>
+  </gazebo> -->
+  <!-- <gazebo reference="LiCAS_A1_q2_1">
+    <provideFeedback>true</provideFeedback>
+  </gazebo>
+  <gazebo>
+    <plugin name="LiCAS_A1_q2_1_sensor" filename="libgazebo_ros_ft_sensor.so">
+      <updateRate>100.0</updateRate>
+      <topicName>LiCAS_A1_q2_1_sensor</topicName>
+      <jointName>LiCAS_A1_q2_1</jointName>
+    </plugin>
+  </gazebo> -->
+  <!-- <gazebo reference="LiCAS_A1_q2_2">
+    <provideFeedback>true</provideFeedback>
+  </gazebo>
+  <gazebo>
+    <plugin name="LiCAS_A1_q2_2_sensor" filename="libgazebo_ros_ft_sensor.so">
+      <updateRate>100.0</updateRate>
+      <topicName>LiCAS_A1_q2_2_sensor</topicName>
+      <jointName>LiCAS_A1_q2_2</jointName>
+    </plugin>
+  </gazebo> -->
+  <!-- <gazebo reference="LiCAS_A1_q2_3">
+    <provideFeedback>true</provideFeedback>
+  </gazebo>
+  <gazebo>
+    <plugin name="LiCAS_A1_q2_3_sensor" filename="libgazebo_ros_ft_sensor.so">
+      <updateRate>100.0</updateRate>
+      <topicName>LiCAS_A1_q2_3_sensor</topicName>
+      <jointName>LiCAS_A1_q2_3</jointName>
+    </plugin>
+  </gazebo> -->
+  <!-- <gazebo reference="LiCAS_A1_q2_4">
+    <provideFeedback>true</provideFeedback>
+  </gazebo>
+  <gazebo>
+    <plugin name="LiCAS_A1_q2_4_sensor" filename="libgazebo_ros_ft_sensor.so">
+      <updateRate>100.0</updateRate>
+      <topicName>LiCAS_A1_q2_4_sensor</topicName>
+      <jointName>LiCAS_A1_q2_4</jointName>
+    </plugin>
+  </gazebo> -->
+  <!-- <gazebo>
+    <plugin name="f3d_plugin" filename="libgazebo_ros_f3d.so">
+      <robotNamespace>licasa1</robotNamespace>
+      <bodyName>left_eef_link</bodyName>
+      <topicName>left_eef_link/body_wrench</topicName>
+    </plugin>
+  </gazebo>   -->
 </robot>
