Commit message: Estimator now uses Butterworth transfer function

File: rotors_simulator/rotors_description/urdf/licasa1.xacro (robot description, xacro)
@@ -518,4 +518,16 @@
       <inertia ixx="1e-03" ixy="0.0" ixz="0.0" iyy="1e-03" iyz="0.0" izz="1e-03"/>
     </inertial>
+    <!-- <visual>
+      <origin xyz="0 0 0"/>
+      <geometry>
+        <sphere radius="0.01"/>
+      </geometry>
+    </visual>
+    <collision>
+      <origin xyz="0 0 0"/>
+      <geometry>
+        <sphere radius="0.01"/>
+      </geometry>
+    </collision> -->
   </link>
   <joint name="left_eef_joint" type="fixed">
@@ -530,93 +542,16 @@
       <inertia ixx="1e-03" ixy="0.0" ixz="0.0" iyy="1e-03" iyz="0.0" izz="1e-03"/>
     </inertial>
-  </link>
-  <!-- Enable the Joint Feedback -->
-    <!-- The ft_sensor plugin -->
-  <!-- <gazebo reference="LiCAS_A1_q1_1">
-    <provideFeedback>true</provideFeedback>
-  </gazebo>
-  <gazebo>
-    <plugin name="LiCAS_A1_q1_1_sensor" filename="libgazebo_ros_ft_sensor.so">
-      <updateRate>100.0</updateRate>
-      <topicName>LiCAS_A1_q1_1_sensor</topicName>
-      <jointName>LiCAS_A1_q1_1</jointName>
-    </plugin>
-  </gazebo> -->
-  <!-- <gazebo reference="LiCAS_A1_q1_2">
-    <provideFeedback>true</provideFeedback>
-  </gazebo>
-  <gazebo>
-    <plugin name="LiCAS_A1_q1_2_sensor" filename="libgazebo_ros_ft_sensor.so">
-      <updateRate>100.0</updateRate>
-      <topicName>LiCAS_A1_q1_2_sensor</topicName>
-      <jointName>LiCAS_A1_q1_2</jointName>
-    </plugin>
-  </gazebo> -->
-  <!-- <gazebo reference="LiCAS_A1_q1_3">
-    <provideFeedback>true</provideFeedback>
-  </gazebo>
-  <gazebo>
-    <plugin name="LiCAS_A1_q1_3_sensor" filename="libgazebo_ros_ft_sensor.so">
-      <updateRate>100.0</updateRate>
-      <topicName>LiCAS_A1_q1_3_sensor</topicName>
-      <jointName>LiCAS_A1_q1_3</jointName>
-    </plugin>
-  </gazebo> -->
-  <!-- <gazebo reference="LiCAS_A1_q1_4">
-    <provideFeedback>true</provideFeedback>
-  </gazebo>
-  <gazebo>
-    <plugin name="LiCAS_A1_q1_4_sensor" filename="libgazebo_ros_ft_sensor.so">
-      <updateRate>100.0</updateRate>
-      <topicName>LiCAS_A1_q1_4_sensor</topicName>
-      <jointName>LiCAS_A1_q1_4</jointName>
-    </plugin>
-  </gazebo> -->
-  <!-- <gazebo reference="LiCAS_A1_q2_1">
-    <provideFeedback>true</provideFeedback>
-  </gazebo>
-  <gazebo>
-    <plugin name="LiCAS_A1_q2_1_sensor" filename="libgazebo_ros_ft_sensor.so">
-      <updateRate>100.0</updateRate>
-      <topicName>LiCAS_A1_q2_1_sensor</topicName>
-      <jointName>LiCAS_A1_q2_1</jointName>
-    </plugin>
-  </gazebo> -->
-  <!-- <gazebo reference="LiCAS_A1_q2_2">
-    <provideFeedback>true</provideFeedback>
-  </gazebo>
-  <gazebo>
-    <plugin name="LiCAS_A1_q2_2_sensor" filename="libgazebo_ros_ft_sensor.so">
-      <updateRate>100.0</updateRate>
-      <topicName>LiCAS_A1_q2_2_sensor</topicName>
-      <jointName>LiCAS_A1_q2_2</jointName>
-    </plugin>
-  </gazebo> -->
-  <!-- <gazebo reference="LiCAS_A1_q2_3">
-    <provideFeedback>true</provideFeedback>
-  </gazebo>
-  <gazebo>
-    <plugin name="LiCAS_A1_q2_3_sensor" filename="libgazebo_ros_ft_sensor.so">
-      <updateRate>100.0</updateRate>
-      <topicName>LiCAS_A1_q2_3_sensor</topicName>
-      <jointName>LiCAS_A1_q2_3</jointName>
-    </plugin>
-  </gazebo> -->
-  <!-- <gazebo reference="LiCAS_A1_q2_4">
-    <provideFeedback>true</provideFeedback>
-  </gazebo>
-  <gazebo>
-    <plugin name="LiCAS_A1_q2_4_sensor" filename="libgazebo_ros_ft_sensor.so">
-      <updateRate>100.0</updateRate>
-      <topicName>LiCAS_A1_q2_4_sensor</topicName>
-      <jointName>LiCAS_A1_q2_4</jointName>
-    </plugin>
-  </gazebo> -->
-  <!-- <gazebo>
-    <plugin name="f3d_plugin" filename="libgazebo_ros_f3d.so">
-      <robotNamespace>licasa1</robotNamespace>
-      <bodyName>left_eef_link</bodyName>
-      <topicName>left_eef_link/body_wrench</topicName>
-    </plugin>
-  </gazebo>   -->
+    <!-- <visual>
+      <origin xyz="0 0 0"/>
+      <geometry>
+        <sphere radius="0.01"/>
+      </geometry>
+    </visual>
+    <collision>
+      <origin xyz="0 0 0"/>
+      <geometry>
+        <sphere radius="0.01"/>
+      </geometry>
+    </collision> -->
+  </link>
 </robot>

File: uav-cable-suspended-robots/uav-cable-suspended-robots-ros-pkg/urdf/licasa1_sensor_wall.urdf.xacro (robot description, xacro)
@@ -4,5 +4,5 @@
   <link name="world" />
   <joint name="sensor_wall_base_joint" type="fixed">
-    <origin xyz="2.5 0 0.05" rpy="0 0 0.75"/>
+    <origin xyz="2.5 0 0.05" rpy="0 0 0"/>
     <parent link="world"/>
     <child link="sensor_wall_base"/>
@@ -56,8 +56,8 @@
   <gazebo reference="sensor_wall">
     <material>Gazebo/DarkGrey</material>
-    <mu1>0.5</mu1>
-    <mu2>0.5</mu2>
-    <kp value="1e2" />
-    <kd value="1e2" />
+    <mu1>0.1</mu1>
+    <mu2>0.1</mu2>
+    <kp value="1e3" />
+    <kd value="1e3" />
   </gazebo>
   <!-- Enable the Joint Feedback -->

Commit message: Fixed Estimator, which is now also easier to tune

File: rotors_simulator/rotors_description/urdf/licasa1.xacro (robot description, xacro)
@@ -521,11 +521,11 @@
       <origin xyz="0 0 0"/>
       <geometry>
-        <sphere radius="0.01"/>
-      </geometry>
-    </visual>
-    <collision>
-      <origin xyz="0 0 0"/>
-      <geometry>
-        <sphere radius="0.01"/>
+        <sphere radius="0.02"/>
+      </geometry>
+    </visual>
+    <collision>
+      <origin xyz="0 0 0"/>
+      <geometry>
+        <sphere radius="0.02"/>
       </geometry>
     </collision> -->
@@ -545,11 +545,11 @@
       <origin xyz="0 0 0"/>
       <geometry>
-        <sphere radius="0.01"/>
-      </geometry>
-    </visual>
-    <collision>
-      <origin xyz="0 0 0"/>
-      <geometry>
-        <sphere radius="0.01"/>
+        <sphere radius="0.02"/>
+      </geometry>
+    </visual>
+    <collision>
+      <origin xyz="0 0 0"/>
+      <geometry>
+        <sphere radius="0.02"/>
       </geometry>
     </collision> -->

Commit message: Finalized estimator, implementing shared control

File: rotors_simulator/rotors_description/urdf/licasa1.xacro (robot description, xacro)
@@ -21,6 +21,8 @@
   <xacro:property name="rotor_velocity_slowdown_sim" value="10" />
   <xacro:property name="use_mesh_file" value="true" /> <!-- true -->
-  <xacro:property name="mesh_file" value="package://rotors_description/meshes/firefly.dae" />
-  <xacro:property name="mass" value="20.269" /> <!-- 1.5 [kg] -->
+  <xacro:property name="mesh_file" value="package://rotors_description/meshes/pelican.dae" />
+  <!-- <xacro:property name="mesh_file" value="package://rotors_description/meshes/Assembly_X4.stl" /> -->
+  <xacro:property name="mesh_scale" value="3.1 3.1 1.5" />
+  <xacro:property name="mass" value="20.269" /> <!-- 20.269 [kg] -->
   <xacro:property name="body_width" value="0.6" /> <!-- 0.1 [m] -->
   <xacro:property name="body_height" value="0.24" /> <!-- 0.16 [m] -->
@@ -57,4 +59,5 @@
     use_mesh_file="${use_mesh_file}"
     mesh_file="${mesh_file}"
+    mesh_scale="${mesh_scale}"
     >
     <xacro:insert_block name="body_inertia" />
@@ -518,16 +521,18 @@
       <inertia ixx="1e-03" ixy="0.0" ixz="0.0" iyy="1e-03" iyz="0.0" izz="1e-03"/>
     </inertial>
-    <!-- <visual>
-      <origin xyz="0 0 0"/>
-      <geometry>
-        <sphere radius="0.02"/>
-      </geometry>
-    </visual>
-    <collision>
-      <origin xyz="0 0 0"/>
-      <geometry>
-        <sphere radius="0.02"/>
-      </geometry>
-    </collision> -->
+    <visual>
+      <origin xyz="0 0 0"/>
+      <geometry>
+        <!-- <sphere radius="0.02"/> -->
+        <box size="0.04 0.04 0.04" />
+      </geometry>
+    </visual>
+    <collision>
+      <origin xyz="0 0 0"/>
+      <geometry>
+        <!-- <sphere radius="0.02"/> -->
+        <box size="0.04 0.04 0.04" />
+      </geometry>
+    </collision>
   </link>
   <joint name="left_eef_joint" type="fixed">
@@ -542,16 +547,88 @@
       <inertia ixx="1e-03" ixy="0.0" ixz="0.0" iyy="1e-03" iyz="0.0" izz="1e-03"/>
     </inertial>
-    <!-- <visual>
-      <origin xyz="0 0 0"/>
-      <geometry>
-        <sphere radius="0.02"/>
-      </geometry>
-    </visual>
-    <collision>
-      <origin xyz="0 0 0"/>
-      <geometry>
-        <sphere radius="0.02"/>
-      </geometry>
-    </collision> -->
-  </link>
+    <visual>
+      <origin xyz="0 0 0"/>
+      <geometry>
+        <!-- <sphere radius="0.02"/> -->
+        <box size="0.04 0.04 0.04" />
+      </geometry>
+    </visual>
+    <collision>
+      <origin xyz="0 0 0"/>
+      <geometry>
+        <!-- <sphere radius="0.02"/> -->
+        <box size="0.04 0.04 0.04" />
+      </geometry>
+    </collision>
+  </link>
+  <!-- <joint name="right_eef_joint_1" type="revolute">
+    <origin xyz="0 0 0"/>
+    <parent link="right_eef_link"/>
+    <child link="right_eef_link_1"/>
+    <axis xyz="0 0 1"/>
+    <dynamics damping="0.0" friction="0.0"/>
+    <limit effort="10.0" lower="0" upper="0" velocity="6"/>
+  </joint>
+  <link name="right_eef_link_1">
+    <inertial>
+      <origin rpy="0 0 0" xyz="0 0 0"/>
+      <mass value="1e-3" />
+      <inertia ixx="1e-03" ixy="0.0" ixz="0.0" iyy="1e-03" iyz="0.0" izz="1e-03"/>
+    </inertial>
+  </link>
+  <joint name="left_eef_joint_1" type="revolute">
+    <origin xyz="0 0 0"/>
+    <parent link="left_eef_link"/>
+    <child link="left_eef_link_1"/>
+    <axis xyz="0 0 1"/>
+    <dynamics damping="0.0" friction="0.0"/>
+    <limit effort="10.0" lower="0" upper="0" velocity="6"/>
+  </joint>
+  <link name="left_eef_link_1">
+    <inertial>
+      <origin rpy="0 0 0" xyz="0 0 0"/>
+      <mass value="1e-3" />
+      <inertia ixx="1e-03" ixy="0.0" ixz="0.0" iyy="1e-03" iyz="0.0" izz="1e-03"/>
+    </inertial>
+  </link>  -->
+  <gazebo>
+    <plugin name="f3d_plugin" filename="libgazebo_ros_f3d.so">
+      <robotNamespace>licasa1</robotNamespace>
+      <bodyName>left_eef_link</bodyName>
+      <topicName>left_eef_link/body_wrench</topicName>
+    </plugin>
+  </gazebo>
+  <gazebo>
+    <plugin name="f3d_plugin" filename="libgazebo_ros_f3d.so">
+      <robotNamespace>licasa1</robotNamespace>
+      <bodyName>right_eef_link</bodyName>
+      <topicName>right_eef_link/body_wrench</topicName>
+    </plugin>
+  </gazebo>
+  <!-- GRASP PLUGIN -->
+  <!-- <gazebo>
+   <plugin name="gazebo_grasp_fix" filename="libgazebo_grasp_fix.so">
+        <arm>
+           <arm_name>licasa1_arm</arm_name>
+           <palm_link>shoulder_link_y</palm_link>
+           <gripper_link>left_shoulder_roll</gripper_link>
+           <gripper_link>left_shoulder_yaw</gripper_link>
+           <gripper_link>left_elbow_pitch</gripper_link>
+           <gripper_link>left_forearm_link</gripper_link>
+           <gripper_link>left_eef_link</gripper_link>
+           <gripper_link>right_shoulder_roll</gripper_link>
+           <gripper_link>right_shoulder_yaw</gripper_link>
+           <gripper_link>right_elbow_pitch</gripper_link>
+           <gripper_link>right_forearm_link</gripper_link>
+           <gripper_link>right_eef_link</gripper_link>
+        </arm>
+       <forces_angle_tolerance>100</forces_angle_tolerance>
+       <update_rate>4</update_rate>
+       <grip_count_threshold>4</grip_count_threshold>
+       <max_grip_count>8</max_grip_count>
+       <release_tolerance>0.005</release_tolerance>
+       <disable_collisions_on_attach>false</disable_collisions_on_attach>
+       <contact_topic>/licasa1/contact_topic</contact_topic>
+    </plugin>
+</gazebo> -->
 </robot>

File: rotors_simulator/rotors_description/urdf/multirotor_base.xacro (robot description, xacro)
@@ -33,5 +33,5 @@
   <!-- Main multirotor link -->
   <xacro:macro name="multirotor_base_macro"
-    params="robot_namespace mass body_width body_height use_mesh_file mesh_file *inertia">
+    params="robot_namespace mass body_width body_height use_mesh_file mesh_file mesh_scale *inertia">
     <link name="${robot_namespace}/base_link"></link>
     <joint name="${robot_namespace}/base_joint" type="fixed">
@@ -50,5 +50,5 @@
         <geometry>
           <xacro:if value="${use_mesh_file}">
-            <mesh filename="${mesh_file}" scale="1 1 1" />
+            <mesh filename="${mesh_file}" scale="${mesh_scale}" />
           </xacro:if>
           <xacro:unless value="${use_mesh_file}">

File: uav-cable-suspended-robots/uav-cable-suspended-robots-ros-pkg/urdf/licasa1_launchpad.urdf.xacro (robot description, xacro)
@@ -100,4 +100,32 @@
     </collision>
   </link>
+  <gazebo reference="left_launchpad">
+    <material>Gazebo/Turquoise</material>
+    <mu1>0.5</mu1>
+    <mu2>0.5</mu2>
+    <kp value="1e6" />
+    <kd value="1e6" />
+  </gazebo>
+  <gazebo reference="left_launchpad_top">
+    <material>Gazebo/Turquoise</material>
+    <mu1>0.5</mu1>
+    <mu2>0.5</mu2>
+    <kp value="1e6" />
+    <kd value="1e6" />
+  </gazebo>
+  <gazebo reference="right_launchpad">
+    <material>Gazebo/Turquoise</material>
+    <mu1>0.5</mu1>
+    <mu2>0.5</mu2>
+    <kp value="1e6" />
+    <kd value="1e6" />
+  </gazebo>
+  <gazebo reference="right_launchpad_top">
+    <material>Gazebo/Turquoise</material>
+    <mu1>0.5</mu1>
+    <mu2>0.5</mu2>
+    <kp value="1e6" />
+    <kd value="1e6" />
+  </gazebo>
   <!-- <joint name="sensor_wall_base_joint" type="fixed">
     <origin xyz="2.5 0 0.05"/>
